File: solar-ltc4015/LTC4015.kicad_sch (KiCad schematic)
At the start: 51 parts, among them J201 Conn_01x05, Q201 FDMC8327L, Q202 FDMC8030, Q203 DMP4013LFGQ-13, U201 LTC4015EUHF#TRPBF

Commit message: Update layout
Other:
- note added: "LM76002RNPR"
Changed lines of the file:
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@@
 	(generator_version "9.0")
 	(paper "A3")
+	(text "LM76002RNPR"
+		(exclude_from_sim no)
+		(at 70.612 56.896 0)
+		(effects
+			(font
+				(size 1.27 1.27)
+			)
+		)
+	)
 	(text_box "TODO:\nInput/Output filters? C87510\nCan I reduce capacitors for the V_SYS since we are not using that as a power out?\nDo I need to do something do disalbe the couloumb counter on the LTC4015?\nShould I take the power out from the high side of the battery shunt resistor instead of the battery directly?\n"
 		(exclude_from_sim no)
