File: solar-ltc4015/cell_1.kicad_sch (KiCad schematic)
At the start: 12 parts, among them Q301 DMP2040UFDF-7, Q302 Q_PMOS_GSD, Q303 FS8205A_C908265, U301 BQ297xy

Commit message: Update layout
Parts:
- Q302: symbol Device:Q_PMOS_GSD -> Transistor_FET:Q_PMOS_GSD
Changed lines of the file:
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@@
 	)
 	(symbol
-		(lib_id "Device:Q_PMOS_GSD")
+		(lib_id "Transistor_FET:Q_PMOS_GSD")
 		(at 91.44 59.69 0)
 		(mirror x)
@@
 			)
 		)
-		(property "Description" ""
+		(property "Description" "P-MOSFET transistor, gate/source/drain"
 			(at 91.44 59.69 0)
 			(effects
