File: solar-ltc4015/kicadpartsplacer.kicad_pcb (KiCad board)
At the start: 4 copper layers, 177.8 x 207.1 mm, 330 parts, among them J101 Power In, J102 Power OUT, J103 Power OUT, J201 Conn_01x05, Q1001 DMP2040UFDF-7, Q1002 Q_PMOS_GSD, Q1003 FS8205A_C908265, Q1101 DMP2040UFDF-7, Q1102 Q_PMOS_GSD, Q1103 FS8205A_C908265, Q1201 DMP2040UFDF-7, Q1202 Q_PMOS_GSD, Q1203 FS8205A_C908265, Q1301 DMP2040UFDF-7, Q1302 Q_PMOS_GSD, Q1303 FS8205A_C908265, Q1401 DMP2040UFDF-7, Q1402 Q_PMOS_GSD, Q1403 FS8205A_C908265, Q1501 DMP2040UFDF-7, Q1502 Q_PMOS_GSD, Q1503 FS8205A_C908265, Q1601 DMP2040UFDF-7, Q1602 Q_PMOS_GSD, Q1603 FS8205A_C908265, Q1701 DMP2040UFDF-7, Q1702 Q_PMOS_GSD, Q1703 FS8205A_C908265, Q1801 DMP2040UFDF-7, Q1802 Q_PMOS_GSD, Q1803 FS8205A_C908265, Q201 FDMC8327L, Q202 FDMC8030, Q203 DMP4013LFGQ-13, Q301 DMP2040UFDF-7, Q302 Q_PMOS_GSD, Q303 FS8205A_C908265, Q401 DMP2040UFDF-7, Q402 Q_PMOS_GSD, Q403 FS8205A_C908265, Q501 DMP2040UFDF-7, Q502 Q_PMOS_GSD, Q503 FS8205A_C908265, Q601 DMP2040UFDF-7, Q602 Q_PMOS_GSD, Q603 FS8205A_C908265, Q701 DMP2040UFDF-7, Q702 Q_PMOS_GSD, Q703 FS8205A_C908265, Q801 DMP2040UFDF-7, Q802 Q_PMOS_GSD, Q803 FS8205A_C908265, Q901 DMP2040UFDF-7, Q902 Q_PMOS_GSD, Q903 FS8205A_C908265, U1001 BQ297xy, U1101 BQ297xy, U1201 BQ297xy, U1301 BQ297xy, U1401 BQ297xy, U1501 BQ297xy, U1601 BQ297xy, U1701 BQ297xy, U1801 BQ297xy, U201 LTC4015EUHF#TRPBF, U301 BQ297xy, U401 BQ297xy, U501 BQ297xy, U601 BQ297xy, U701 BQ297xy, U801 BQ297xy, U901 BQ297xy

Commit message: Update layout
Parts:
- moved Q1103 254.0 mm to (174.9, -156.5), turned to 0 degrees
- moved Q803 250.7 mm to (174.9, -124.7), turned to 0 degrees
- moved Q603 249.0 mm to (124.9, -156.5), turned to 0 degrees
- moved Q1003 236.8 mm to (162.4, -140.6), turned to 0 degrees
- moved Q703 233.2 mm to (137.4, -124.7), turned to 0 degrees
- moved Q1203 232.0 mm to (174.9, -140.6), turned to 0 degrees
- moved Q1303 212.6 mm to (149.9, -140.6), turned to 0 degrees
- moved Q903 209.8 mm to (124.9, -124.7), turned to 0 degrees
- moved Q1603 206.7 mm to (149.9, -156.5), turned to 0 degrees
- moved Q1803 203.6 mm to (162.4, -156.5), turned to 0 degrees
- moved Q1703 199.3 mm to (137.4, -156.5), turned to 0 degrees
- moved Q1403 198.7 mm to (162.4, -124.7), turned to 0 degrees
- moved Q1503 194.3 mm to (137.4, -140.6), turned to 0 degrees
- moved Q701 181.5 mm to (137.0, -117.6)
- moved R704 181.5 mm to (137.0, -121.0)
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Routing:
- net /cell_2/BAT-: track 68.1 -> 69.2 mm
