File: solar-ltc4015/solar-ltc4015.kicad_pcb (KiCad board)
At the start: 4 copper layers, 177.8 x 207.1 mm, 330 parts, among them J101 Power In, J102 Power OUT, J103 Power OUT, J201 Conn_01x05, Q1001 DMP2040UFDF-7, Q1002 Q_PMOS_GSD, Q1003 FS8205A_C908265, Q1101 DMP2040UFDF-7, Q1102 Q_PMOS_GSD, Q1103 FS8205A_C908265, Q1201 DMP2040UFDF-7, Q1202 Q_PMOS_GSD, Q1203 FS8205A_C908265, Q1301 DMP2040UFDF-7, Q1302 Q_PMOS_GSD, Q1303 FS8205A_C908265, Q1401 DMP2040UFDF-7, Q1402 Q_PMOS_GSD, Q1403 FS8205A_C908265, Q1501 DMP2040UFDF-7, Q1502 Q_PMOS_GSD, Q1503 FS8205A_C908265, Q1601 DMP2040UFDF-7, Q1602 Q_PMOS_GSD, Q1603 FS8205A_C908265, Q1701 DMP2040UFDF-7, Q1702 Q_PMOS_GSD, Q1703 FS8205A_C908265, Q1801 DMP2040UFDF-7, Q1802 Q_PMOS_GSD, Q1803 FS8205A_C908265, Q201 FDMC8327L, Q202 FDMC8030, Q203 DMP4013LFGQ-13, Q301 DMP2040UFDF-7, Q302 Q_PMOS_GSD, Q303 FS8205A_C908265, Q401 DMP2040UFDF-7, Q402 Q_PMOS_GSD, Q403 FS8205A_C908265, Q501 DMP2040UFDF-7, Q502 Q_PMOS_GSD, Q503 FS8205A_C908265, Q601 DMP2040UFDF-7, Q602 Q_PMOS_GSD, Q603 FS8205A_C908265, Q701 DMP2040UFDF-7, Q702 Q_PMOS_GSD, Q703 FS8205A_C908265, Q801 DMP2040UFDF-7, Q802 Q_PMOS_GSD, Q803 FS8205A_C908265, Q901 DMP2040UFDF-7, Q902 Q_PMOS_GSD, Q903 FS8205A_C908265, U1001 BQ297xy, U1101 BQ297xy, U1201 BQ297xy, U1301 BQ297xy, U1401 BQ297xy, U1501 BQ297xy, U1601 BQ297xy, U1701 BQ297xy, U1801 BQ297xy, U201 LTC4015EUHF#TRPBF, U301 BQ297xy, U401 BQ297xy, U501 BQ297xy, U601 BQ297xy, U701 BQ297xy, U801 BQ297xy, U901 BQ297xy

Commit message: Update layout
Parts:
- removed REF**: 2.2k, Resistor_SMD:R_0402_1005Metric
- removed REF**: BQ297xy, cacophony-library:WSON-6_1.5x1.5mm_P0.5mm
- removed REF**: 100k, Resistor_SMD:R_0402_1005Metric
- removed REF**: DMP2040UFDF-7, Package_DFN_QFN:Diodes_UDFN2020-6_Type-F
- removed REF**: Q_PMOS_GSD, cacophony-library:SOT-523
- removed REF**: 22mΩ, Resistor_SMD:R_0805_2012Metric
- removed REF**: MY-18650-05-J, cacophony-library:BAT-TH_MY-18650-05-J
- removed REF**: FS8205A_C908265, Package_TO_SOT_SMD:SOT-23-6
- removed REF** (x2): 4.7M, Resistor_SMD:R_0402_1005Metric
- removed REF**: 330Ω, Resistor_SMD:R_0402_1005Metric
- removed REF**: 1M, Resistor_SMD:R_0402_1005Metric
- removed REF** (x2): MountingHole, cacophony-library:MountingHole_3.2mm_no_bolt_head
- removed REF**: 100nF, Resistor_SMD:R_0402_1005Metric
- moved R304 402.9 mm to (-79.0, 28.4), turned to 90 degrees
- moved R704 400.3 mm to (-40.4, 28.4), turned to 90 degrees
- moved R305 397.7 mm to (-80.8, 27.2)
- moved U301 397.2 mm to (-79.3, 21.3)
- moved C301 396.0 mm to (-78.9, 19.3), turned to 90 degrees
- moved R504 395.9 mm to (-59.7, 28.4), turned to 90 degrees
- moved R306 394.8 mm to (-81.0, 21.4), turned to 90 degrees
- moved R705 394.8 mm to (-42.2, 27.2)
- moved R303 394.3 mm to (-79.9, 18.6), turned to -90 degrees
- moved U701 394.1 mm to (-40.7, 21.3)
- moved R307 393.1 mm to (-80.9, 19.2), turned to 90 degrees
- moved C701 393.1 mm to (-40.3, 19.3), turned to 90 degrees
- moved R706 391.5 mm to (-42.4, 21.4), turned to 90 degrees
- moved R703 391.1 mm to (-41.3, 18.6), turned to -90 degrees
- moved R505 391.0 mm to (-61.5, 27.2)
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Routing:
- net (no net): track 114.0 -> 0.00 mm, vias 3 -> 0
- net Net-(U201-NTC): track 17.3 -> 104.3 mm, vias 0 -> 2
- net /cell_1/BAT-: track 0.00 -> 79.0 mm
- net /cell_9/BAT-: track 0.00 -> 69.2 mm
- net /cell_8/BAT-: track 0.00 -> 69.2 mm
- net /cell_7/BAT-: track 0.00 -> 69.2 mm
- net /cell_6/BAT-: track 0.00 -> 69.2 mm
- net /cell_5/BAT-: track 0.00 -> 69.2 mm
- net /cell_4/BAT-: track 0.00 -> 69.2 mm
- net /cell_3/BAT-: track 0.00 -> 69.2 mm
- net /cell_14/BAT-: track 0.00 -> 69.2 mm
- net /cell_13/BAT-: track 0.00 -> 69.2 mm
- net /cell_10/BAT-: track 0.00 -> 69.2 mm
- net /cell_15/BAT-: track 0.00 -> 69.2 mm
- net /cell_12/BAT-: track 0.00 -> 69.2 mm
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- added copper zone on F.Cu, net /GND_IN_FILTERED
- added copper zone on In2.Cu, net /GND_OUT_FILTERED
- added copper zone on In2.Cu, net /V_BAT_FILTERED
Other:
- board size 177.8 x 207.1 mm -> 175 x 85 mm
