File: solar-ltc4015/solar-ltc4015.kicad_sch (KiCad schematic)
At the start: 72 parts, among them J101 Power In, J102 Power OUT, J103 Power OUT

Commit message: Update layout
Changed lines of the file:
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@@
 	(text "C2915633"
 		(exclude_from_sim no)
-		(at 279.654 119.38 0)
+		(at 288.798 119.888 0)
 		(effects
 			(font
@@
 		)
 		(instances
-			(project "solar-ltc4015"
+			(project "kicadpartsplacer"
 				(path "/822b745e-d66e-4222-a6d2-360780548724"
 					(page "c4")
@@
 		)
 		(instances
-			(project "solar-ltc4015"
+			(project "kicadpartsplacer"
 				(path "/822b745e-d66e-4222-a6d2-360780548724"
 					(page "c1")
@@
 		)
 		(instances
-			(project "solar-ltc4015"
+			(project "kicadpartsplacer"
 				(path "/822b745e-d66e-4222-a6d2-360780548724"
 					(page "c7")
@@
 		)
 		(instances
-			(project "solar-ltc4015"
+			(project "kicadpartsplacer"
 				(path "/822b745e-d66e-4222-a6d2-360780548724"
 					(page "c15")
@@
 		)
 		(instances
-			(project "solar-ltc4015"
+			(project "kicadpartsplacer"
 				(path "/822b745e-d66e-4222-a6d2-360780548724"
 					(page "c13")
@@
 		)
 		(instances
-			(project "solar-ltc4015"
+			(project "kicadpartsplacer"
 				(path "/822b745e-d66e-4222-a6d2-360780548724"
 					(page "c5")
@@
 		)
 		(instances
-			(project "solar-ltc4015"
+			(project "kicadpartsplacer"
 				(path "/822b745e-d66e-4222-a6d2-360780548724"
 					(page "c14")
@@
 		)
 		(instances
-			(project "solar-ltc4015"
+			(project "kicadpartsplacer"
 				(path "/822b745e-d66e-4222-a6d2-360780548724"
 					(page "c16")
@@
 		)
 		(instances
-			(project "solar-ltc4015"
+			(project "kicadpartsplacer"
 				(path "/822b745e-d66e-4222-a6d2-360780548724"
 					(page "c9")
@@
 		)
 		(instances
-			(project "solar-ltc4015"
+			(project "kicadpartsplacer"
 				(path "/822b745e-d66e-4222-a6d2-360780548724"
 					(page "2")
@@
 		)
 		(instances
-			(project "solar-ltc4015"
+			(project "kicadpartsplacer"
 				(path "/822b745e-d66e-4222-a6d2-360780548724"
 					(page "c2")
@@
 		)
 		(instances
-			(project "solar-ltc4015"
+			(project "kicadpartsplacer"
 				(path "/822b745e-d66e-4222-a6d2-360780548724"
 					(page "c11")
@@
 		)
 		(instances
-			(project "solar-ltc4015"
+			(project "kicadpartsplacer"
 				(path "/822b745e-d66e-4222-a6d2-360780548724"
 					(page "c3")
@@
 		)
 		(instances
-			(project "solar-ltc4015"
+			(project "kicadpartsplacer"
 				(path "/822b745e-d66e-4222-a6d2-360780548724"
 					(page "c8")
@@
 		)
 		(instances
-			(project "solar-ltc4015"
+			(project "kicadpartsplacer"
 				(path "/822b745e-d66e-4222-a6d2-360780548724"
 					(page "c10")
@@
 		)
 		(instances
-			(project "solar-ltc4015"
+			(project "kicadpartsplacer"
 				(path "/822b745e-d66e-4222-a6d2-360780548724"
 					(page "c12")
@@
 		)
 		(instances
-			(project "solar-ltc4015"
+			(project "kicadpartsplacer"
 				(path "/822b745e-d66e-4222-a6d2-360780548724"
 					(page "c6")
