File: solar-BQ25798/LTC4015.kicad_sch (KiCad schematic)
At the start: 51 parts, among them J201 Conn_01x05, Q201 FDMC8327L, Q202 FDMC8030, Q203 DMP4013LFGQ-13, U201 LTC4015EUHF#TRPBF

Commit message: BQ25798 WIP
Parts:
- J1801: renamed from J201; now left out of the parts list
- R1810: renamed from R204; value R -> 100k; LCSC Part (none) -> C25741
- renumbered C204 to C1801, C206 to C1802, C207 to C1803, C208 to C1804, C218 to C1805, C220 to C1806, C223 to C1807, C225 to C1808, C227 to C1809, C209 to C1810, C221 to C1811, C224 to C1812, C226 to C1813, C228 to C1814, C205 to C1815, C213 to C1816, C216 to C1817, C215 to C1818, C217 to C1819, C212 to C1820, C210 to C1821, C214 to C1822, C211 to C1823, C219 to C1824, C222 to C1825, C203 to C1826, C201 to C1827, C202 to C1828, D201 to D1801, JP201 to JP1801, JP204 to JP1802, JP202 to JP1803, JP203 to JP1804, L201 to L1801, Q201 to Q1801, Q203 to Q1802, Q202 to Q1803, R210 to R1801, R205 to R1802, R206 to R1803, R201 to R1804, R203 to R1805, R207 to R1806, R211 to R1807, R202 to R1808, R212 to R1809, R208 to R1811, TH201 to TH1801, U201 to U1801
