File: solar-BQ25798/cell_S1_3.kicad_sch (KiCad schematic)
At the start: 12 parts, among them Q301 DMP2040UFDF-7, Q302 Q_PMOS_GSD, Q303 FS8205A_C908265, U301 BQ297xy

Commit message: BQ25798 WIP
Parts:
- R501: renamed from R301; LCSC Part (none) -> C26083
- R502: renamed from R302; LCSC Part (none) -> C25741
- R505: renamed from R305; LCSC Part C23163 -> C208994
- R506: renamed from R306; LCSC Part C23163 -> C208994
- renumbered C301 to C501, Q301 to Q501, Q302 to Q502, Q303 to Q503, R303 to R503, R304 to R504, R307 to R507, U301 to U501
Changed lines of the file:
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@@
 	(generator_version "9.0")
 	(paper "A4")
+	(text_box "~30mΩ at 3.7V"
+		(exclude_from_sim no)
+		(at 177.8 114.3 0)
+		(size 16.51 3.81)
+		(margins 0.9525 0.9525 0.9525 0.9525)
+		(stroke
+			(width 0)
+			(type solid)
+		)
+		(fill
+			(type none)
+		)
+		(effects
+			(font
+				(size 1.27 1.27)
+			)
+			(justify left top)
+		)
+	)
+	(text_box "~40mV at 3.7V"
+		(exclude_from_sim no)
+		(at 71.12 13.97 0)
+		(size 17.78 3.81)
+		(margins 0.9525 0.9525 0.9525 0.9525)
+		(stroke
+			(width 0)
+			(type solid)
+		)
+		(fill
+			(type none)
+		)
+		(effects
+			(font
+				(size 1.27 1.27)
+			)
+			(justify left top)
+		)
+	)
 	(junction
 		(at 186.69 82.55)
@@
 		(dnp no)
 		(fields_autoplaced yes)
-		(property "Reference" "Q301"
+		(property "Reference" "Q501"
 			(at 77.47 31.75 90)
 			(effects
@@
 				(path "/822b745e-d66e-4222-a6d2-360780548724/6cd84410-936a-4acf-ac1c-6f538e56c498"
 					(reference "Q1601")
-					(unit 1)
-				)
-				(path "/822b745e-d66e-4222-a6d2-360780548724/7c20caf5-fe9e-4a5c-bac2-68cabfeaae32"
-					(reference "Q1801")
 					(unit 1)
 				)
@@
 		(dnp no)
 		(fields_autoplaced yes)
-		(property "Reference" "#PWR03001"
+		(property "Reference" "#PWR0401"
 			(at 227.33 49.53 0)
 			(effects
@@
 				(path "/822b745e-d66e-4222-a6d2-360780548724/6cd84410-936a-4acf-ac1c-6f538e56c498"
 					(reference "#PWR02901")
-					(unit 1)
-				)
-				(path "/822b745e-d66e-4222-a6d2-360780548724/7c20caf5-fe9e-4a5c-bac2-68cabfeaae32"
-					(reference "#PWR01801")
 					(unit 1)
 				)
@@
 		(dnp no)
 		(fields_autoplaced yes)
-		(property "Reference" "R302"
+		(property "Reference" "R502"
 			(at 96.52 73.6599 0)
 			(effects
@@
 		)
 		(property "Description" "Resistor"
+			(at 93.98 74.93 0)
+			(effects
+				(font
+					(size 1.27 1.27)
+				)
+				(hide yes)
+			)
+		)
+		(property "LCSC Part" "C25741"
 			(at 93.98 74.93 0)
 			(effects
@@
 				(path "/822b745e-d66e-4222-a6d2-360780548724/6cd84410-936a-4acf-ac1c-6f538e56c498"
 					(reference "R1602")
-					(unit 1)
-				)
-				(path "/822b745e-d66e-4222-a6d2-360780548724/7c20caf5-fe9e-4a5c-bac2-68cabfeaae32"
-					(reference "R1802")
 					(unit 1)
 				)
@@
 		(dnp no)
 		(fields_autoplaced yes)
-		(property "Reference" "R306"
+		(property "Reference" "R506"
 			(at 200.66 99.0599 0)
 			(effects
@@
 			)
 		)
-		(property "LCSC Part" "C23163"
+		(property "LCSC Part" "C208994"
 			(at 198.12 100.33 0)
 			(effects
@@
 				(path "/822b745e-d66e-4222-a6d2-360780548724/6cd84410-936a-4acf-ac1c-6f538e56c498"
 					(reference "R1606")
-					(unit 1)
-				)
-				(path "/822b745e-d66e-4222-a6d2-360780548724/7c20caf5-fe9e-4a5c-bac2-68cabfeaae32"
-					(reference "R1806")
 					(unit 1)
 				)
@@
 		(dnp no)
 		(fields_autoplaced yes)
-		(property "Reference" "#PWR03002"
+		(property "Reference" "#PWR0402"
 			(at 227.33 119.38 0)
 			(effects
@@
 				(path "/822b745e-d66e-4222-a6d2-360780548724/6cd84410-936a-4acf-ac1c-6f538e56c498"
 					(reference "#PWR02902")
-					(unit 1)
-				)
-				(path "/822b745e-d66e-4222-a6d2-360780548724/7c20caf5-fe9e-4a5c-bac2-68cabfeaae32"
-					(reference "#PWR01802")
 					(unit 1)
 				)
@@
 		(dnp no)
 		(fields_autoplaced yes)
-		(property "Reference" "R307"
+		(property "Reference" "R507"
 			(at 215.9 99.0599 0)
 			(effects
@@
 				(path "/822b745e-d66e-4222-a6d2-360780548724/6cd84410-936a-4acf-ac1c-6f538e56c498"
 					(reference "R1607")
-					(unit 1)
-				)
-				(path "/822b745e-d66e-4222-a6d2-360780548724/7c20caf5-fe9e-4a5c-bac2-68cabfeaae32"
-					(reference "R1807")
 					(unit 1)
 				)
@@
 		(dnp no)
 		(fields_autoplaced yes)
-		(property "Reference" "U301"
+		(property "Reference" "U501"
 			(at 160.02 57.15 0)
 			(effects
@@
 				(path "/822b745e-d66e-4222-a6d2-360780548724/6cd84410-936a-4acf-ac1c-6f538e56c498"
 					(reference "U1601")
-					(unit 1)
-				)
-				(path "/822b745e-d66e-4222-a6d2-360780548724/7c20caf5-fe9e-4a5c-bac2-68cabfeaae32"
-					(reference "U1801")
 					(unit 1)
 				)
@@
 		(dnp no)
 		(fields_autoplaced yes)
-		(property "Reference" "R304"
+		(property "Reference" "R504"
 			(at 157.48 105.41 90)
 			(effects
@@
 				(path "/822b745e-d66e-4222-a6d2-360780548724/6cd84410-936a-4acf-ac1c-6f538e56c498"
 					(reference "R1604")
-					(unit 1)
-				)
-				(path "/822b745e-d66e-4222-a6d2-360780548724/7c20caf5-fe9e-4a5c-bac2-68cabfeaae32"
-					(reference "R1804")
 					(unit 1)
 				)
@@
 		(on_board yes)
 		(dnp no)
-		(property "Reference" "Q302"
+		(property "Reference" "Q502"
 			(at 100.1268 59.69 90)
 			(effects
@@
 				(path "/822b745e-d66e-4222-a6d2-360780548724/6cd84410-936a-4acf-ac1c-6f538e56c498"
 					(reference "Q1602")
-					(unit 1)
-				)
-				(path "/822b745e-d66e-4222-a6d2-360780548724/7c20caf5-fe9e-4a5c-bac2-68cabfeaae32"
-					(reference "Q1802")
 					(unit 1)
 				)
@@
 		(dnp no)
 		(fields_autoplaced yes)
-		(property "Reference" "C301"
+		(property "Reference" "C501"
 			(at 135.89 67.3162 0)
 			(effects
@@
 				(path "/822b745e-d66e-4222-a6d2-360780548724/6cd84410-936a-4acf-ac1c-6f538e56c498"
 					(reference "C1601")
-					(unit 1)
-				)
-				(path "/822b745e-d66e-4222-a6d2-360780548724/7c20caf5-fe9e-4a5c-bac2-68cabfeaae32"
-					(reference "C1801")
 					(unit 1)
 				)
@@
 		(dnp no)
 		(fields_autoplaced yes)
-		(property "Reference" "R303"
+		(property "Reference" "R503"
 			(at 135.89 54.6099 0)
 			(effects
@@
 				(path "/822b745e-d66e-4222-a6d2-360780548724/6cd84410-936a-4acf-ac1c-6f538e56c498"
 					(reference "R1603")
-					(unit 1)
-				)
-				(path "/822b745e-d66e-4222-a6d2-360780548724/7c20caf5-fe9e-4a5c-bac2-68cabfeaae32"
-					(reference "R1803")
 					(unit 1)
 				)
@@
 		(dnp no)
 		(fields_autoplaced yes)
-		(property "Reference" "R301"
+		(property "Reference" "R501"
 			(at 77.47 20.32 90)
 			(effects
@@
 		(property "Description" "Resistor"
 			(at 77.47 26.67 0)
+			(effects
+				(font
+					(size 1.27 1.27)
+				)
+				(hide yes)
+			)
+		)
+		(property "LCSC Part" "C26083"
+			(at 77.47 26.67 90)
 			(effects
 				(font
@@
 				(path "/822b745e-d66e-4222-a6d2-360780548724/6cd84410-936a-4acf-ac1c-6f538e56c498"
 					(reference "R1601")
-					(unit 1)
-				)
-				(path "/822b745e-d66e-4222-a6d2-360780548724/7c20caf5-fe9e-4a5c-bac2-68cabfeaae32"
-					(reference "R1801")
 					(unit 1)
 				)
@@
 		(on_board yes)
 		(dnp no)
-		(property "Reference" "Q303"
+		(property "Reference" "Q503"
 			(at 190.5 96.5199 90)
 			(effects
@@
 				(path "/822b745e-d66e-4222-a6d2-360780548724/6cd84410-936a-4acf-ac1c-6f538e56c498"
 					(reference "Q1603")
-					(unit 1)
-				)
-				(path "/822b745e-d66e-4222-a6d2-360780548724/7c20caf5-fe9e-4a5c-bac2-68cabfeaae32"
-					(reference "Q1803")
 					(unit 1)
 				)
@@
 		(dnp no)
 		(fields_autoplaced yes)
-		(property "Reference" "R305"
+		(property "Reference" "R505"
 			(at 168.91 97.7899 0)
 			(effects
@@
 			)
 		)
-		(property "LCSC Part" "C23163"
+		(property "LCSC Part" "C208994"
 			(at 166.37 99.06 0)
 			(effects
@@
 					(unit 1)
 				)
-				(path "/822b745e-d66e-4222-a6d2-360780548724/7c20caf5-fe9e-4a5c-bac2-68cabfeaae32"
-					(reference "R1805")
-					(unit 1)
-				)
