File: solar-BQ25798/solar-BQ25798.kicad_pcb (KiCad board)
At the start: 4 copper layers, 175 x 85 mm, 345 parts, among them J101 Power In, J102 Power OUT, J103 Power OUT, J1701 Conn_01x02, J1901 Conn_01x04, Q1001 DMP2040UFDF-7, Q1002 Q_PMOS_GSD, Q1003 FS8205A_C908265, Q101 DMP4013LFGQ-13, Q1101 DMP2040UFDF-7, Q1102 Q_PMOS_GSD, Q1103 FS8205A_C908265, Q1201 DMP2040UFDF-7, Q1202 Q_PMOS_GSD, Q1203 FS8205A_C908265, Q1301 DMP2040UFDF-7, Q1302 Q_PMOS_GSD, Q1303 FS8205A_C908265, Q1401 DMP2040UFDF-7, Q1402 Q_PMOS_GSD, Q1403 FS8205A_C908265, Q1501 DMP2040UFDF-7, Q1502 Q_PMOS_GSD, Q1503 FS8205A_C908265, Q1601 DMP2040UFDF-7, Q1602 Q_PMOS_GSD, Q1603 FS8205A_C908265, Q1701 CSD17581Q3A, Q1702 CSD17581Q3A, Q1801 CSD17581Q3A, Q1802 CSD17581Q3A, Q1803 Q_PMOS_GSD, Q201 DMP2040UFDF-7, Q202 Q_PMOS_GSD, Q203 FS8205A_C908265, Q301 DMP2040UFDF-7, Q302 Q_PMOS_GSD, Q303 FS8205A_C908265, Q401 DMP2040UFDF-7, Q402 Q_PMOS_GSD, Q403 FS8205A_C908265, Q501 DMP2040UFDF-7, Q502 Q_PMOS_GSD, Q503 FS8205A_C908265, Q601 DMP2040UFDF-7, Q602 Q_PMOS_GSD, Q603 FS8205A_C908265, Q701 DMP2040UFDF-7, Q702 Q_PMOS_GSD, Q703 FS8205A_C908265, Q801 DMP2040UFDF-7, Q802 Q_PMOS_GSD, Q803 FS8205A_C908265, Q901 DMP2040UFDF-7, Q902 Q_PMOS_GSD, Q903 FS8205A_C908265, U1001 BQ297xy, U1101 BQ297xy, U1201 BQ297xy, U1301 BQ297xy, U1401 BQ297xy, U1501 BQ297xy, U1601 BQ297xy, U1701 BQ25798RQMR, U1702 HT75xx-1-SOT89, U1901 ATtiny1616-M, U2 BQ76920PW, U201 BQ297xy, U301 BQ297xy, U401 BQ297xy, U501 BQ297xy, U601 BQ297xy, U701 BQ297xy, U801 BQ297xy, U901 BQ297xy

Commit message: BQ25798 WIP
Parts:
- added BUZZER1901: MLT-7525, cacophony-library:BUZ-SMD_4P-L7.5-W7.5-P7.59-TL, F.Cu at (126.9, -9.90)
- added C1901: 1uF, Capacitor_SMD:C_0402_1005Metric, F.Cu at (131.2, -2.16)
- added C1902: 10uF, Capacitor_SMD:C_0603_1608Metric, F.Cu at (127.8, -3.88)
- added R1901: 180Ω, Resistor_SMD:R_0402_1005Metric, F.Cu at (131.3, -4.14)
- added U1901: AHT20_C2757850, cacophony-library:SENSOR-SMD_L3.0-W3.0-P1.00-BR, F.Cu at (123.2, -2.91)
- F101, F102: value 8A -> 4A; footprint Fuse:Fuse_1206_3216Metric -> cacophony-library:FUSE-SMD_2410F4A250V
- Q1001, Q1101, Q1201, Q1301, Q1401, Q1501, Q1601, Q201, Q301, Q401, Q501, Q601, Q701, Q801, Q901: value DMP2040UFDF-7 -> DMP2035U-7; footprint Package_DFN_QFN:Diodes_UDFN2020-6_Type-F -> Package_TO_SOT_SMD:SOT-23
- Q1701, Q1702: value CSD17581Q3A -> CSD17578Q3A
- Q1801: renamed from Q1802; value CSD17581Q3A -> CSD17578Q3A
- Q1803: renamed from Q1801; value CSD17581Q3A -> CSD17578Q3A
- moved Q301 201.3 mm to (115.0, 48.6)
- moved Q201 189.8 mm to (101.1, 42.1)
- moved Q501 186.5 mm to (115.0, 55.0)
- moved Q401 181.1 mm to (101.1, 61.5)
- moved Q601 170.6 mm to (108.1, 61.5)
- moved Q701 155.6 mm to (121.9, 55.0), turned to 0 degrees
- moved Q801 138.9 mm to (121.9, 42.1), turned to 0 degrees
- moved Q901 121.9 mm to (108.1, 48.6), turned to 0 degrees
- moved Q1201 117.7 mm to (115.0, 42.1)
- moved Q1101 112.5 mm to (115.0, 61.5), turned to 0 degrees
- moved Q1301 109.2 mm to (108.1, 42.1)
- moved Q1001 108.2 mm to (108.1, 55.0), turned to 0 degrees
- moved Q1401 104.0 mm to (101.1, 55.0)
- moved Q1601 99.7 mm to (121.9, 48.6)
- moved Q1501 96.4 mm to (101.1, 48.6)
- renumbered BAT_N106 to BAT_N102, BAT_N111 to BAT_N103, BAT_N102 to BAT_N104, BAT_N107 to BAT_N105, BAT_N112 to BAT_N106, BAT_N103 to BAT_N107, BAT_N113 to BAT_N109, BAT_N104 to BAT_N110, BAT_N109 to BAT_N111, BAT_N114 to BAT_N112, BAT_N105 to BAT_N113, BAT_N110 to BAT_N114, BAT_P106 to BAT_P102, BAT_P111 to BAT_P103, BAT_P102 to BAT_P104, BAT_P107 to BAT_P105, BAT_P112 to BAT_P106, BAT_P103 to BAT_P107, BAT_P113 to BAT_P109, BAT_P104 to BAT_P110, BAT_P109 to BAT_P111, BAT_P114 to BAT_P112, BAT_P105 to BAT_P113, BAT_P110 to BAT_P114, C1708 to C1701, C1722 to C1702, C1721 to C1703, C1705 to C1704, C1706 to C1705, C1707 to C1706, C1715 to C1707, C1718 to C1708, C1719 to C1710, C1723 to C1711, C1710 to C1712, C1711 to C1713, C1712 to C1714, C1713 to C1715, C1701 to C1716, C1714 to C1717, C1720 to C1718, C1702 to C1719, C1703 to C1720, C1716 to C1721, C1704 to C1722, C1717 to C1723, C6 to C1801, C1803 to C1802, C3 to C1803, C2 to C1804, C1 to C1805, C4 to C1806, C5 to C1807, C1801 to C1808, C1802 to C1809, C7 to C1810, C8 to C1811, C10 to C1812, C9 to C1813, C1901 to C1903, D1702 to D1701, D1703 to D1702, D1701 to D1703, D1802 to D1801, H104 to H102, H107 to H103, H110 to H104, H113 to H105, H116 to H106, H119 to H107, H122 to H108, H125 to H109, H127 to H110, H129 to H111, H131 to H112, H102 to H113, H105 to H114, H108 to H115, H111 to H116, H114 to H117, H117 to H118, H120 to H119, H123 to H120, H126 to H121, H128 to H122, H130 to H123, H132 to H124, H103 to H125, H106 to H126, H109 to H127, H112 to H128, H115 to H129, H118 to H130, H121 to H131, H124 to H132, Q1803 to Q1802, R1003 to R1002, R1002 to R1003, R1007 to R1004, R1004 to R1005, R1005 to R1006, R1006 to R1007, R1103 to R1102, R1102 to R1103, R1107 to R1104, R1104 to R1105, R1105 to R1106, R1106 to R1107, R1203 to R1202, R1202 to R1203, R1207 to R1204, R1204 to R1205, R1205 to R1206, R1206 to R1207, R1303 to R1302, R1302 to R1303, R1307 to R1304, R1304 to R1305, R1305 to R1306, R1306 to R1307, R1403 to R1402, R1402 to R1403, R1407 to R1404, R1404 to R1405, R1405 to R1406, R1406 to R1407, R1503 to R1502, R1502 to R1503, R1507 to R1504, R1504 to R1505, R1505 to R1506, R1506 to R1507, R1603 to R1602, R1602 to R1603, R1607 to R1604, R1604 to R1605, R1605 to R1606, R1606 to R1607, R1704 to R1701, R1710 to R1702, R1711 to R1703, R1706 to R1704, R1701 to R1705, R1707 to R1706, R1702 to R1707, R1703 to R1708, R1705 to R1710, R6 to R1801, R5 to R1802, R4 to R1803, R3 to R1804, R2 to R1805, R1 to R1806, R1801 to R1807, R211 to R1808, R1802 to R1809, R1803 to R1810, R7 to R1811, R1805 to R1812, R1804 to R1813, R9 to R1814, R1901 to R1902, R1902 to R1903, R203 to R202, R202 to R203, R207 to R204, R204 to R205, R205 to R206, R206 to R207, R303 to R302, R302 to R303, R307 to R304, R304 to R305, R305 to R306, R306 to R307, R403 to R402, R402 to R403, R407 to R404, R404 to R405, R405 to R406, R406 to R407, R503 to R502, R502 to R503, R507 to R504, R504 to R505, R505 to R506, R506 to R507, R603 to R602, R602 to R603, R607 to R604, R604 to R605, R605 to R606, R606 to R607, R703 to R702, R702 to R703, R707 to R704, R704 to R705, R705 to R706, R706 to R707, R803 to R802, R802 to R803, R807 to R804, R804 to R805, R805 to R806, R806 to R807, R903 to R902, R902 to R903, R907 to R904, R904 to R905, R905 to R906, R906 to R907, TP1910 to TP1901, TP1909 to TP1902, TP1908 to TP1903, TP1907 to TP1904, TP1906 to TP1905, TP1905 to TP1906, TP1904 to TP1907, TP1903 to TP1908, U1702 to U1701, U1701 to U1702, U2 to U1801, U1901 to U1902
Connections:
- Q1001 pad 1: /cell_S1_9/CELL+ -> Net-(Q1001-G)
- Q1001 pad 2: /cell_S1_9/CELL+ -> CELL_2_POSITIVE
- Q1001 pad 3: Net-(Q1001-G) -> /cell_S1_9/CELL+
- Q1101 pad 1: /cell_S1_10/CELL+ -> Net-(Q1101-G)
- Q1101 pad 2: /cell_S1_10/CELL+ -> CELL_2_POSITIVE
- Q1101 pad 3: Net-(Q1101-G) -> /cell_S1_10/CELL+
- Q1201 pad 1: /cell_S1_11/CELL+ -> Net-(Q1201-G)
- Q1201 pad 2: /cell_S1_11/CELL+ -> CELL_1_POSITIVE
- Q1201 pad 3: Net-(Q1201-G) -> /cell_S1_11/CELL+
- Q1301 pad 1: /cell_S1_12/CELL+ -> Net-(Q1301-G)
- Q1301 pad 2: /cell_S1_12/CELL+ -> CELL_1_POSITIVE
- Q1301 pad 3: Net-(Q1301-G) -> /cell_S1_12/CELL+
- Q1401 pad 1: /cell_S1_13/CELL+ -> Net-(Q1401-G)
- Q1401 pad 2: /cell_S1_13/CELL+ -> CELL_1_POSITIVE
- Q1401 pad 3: Net-(Q1401-G) -> /cell_S1_13/CELL+
- Q1501 pad 1: /cell_S1_14/CELL+ -> Net-(Q1501-G)
- Q1501 pad 2: /cell_S1_14/CELL+ -> CELL_1_POSITIVE
- Q1501 pad 3: Net-(Q1501-G) -> /cell_S1_14/CELL+
- Q1601 pad 1: /cell_S1_15/CELL+ -> Net-(Q1601-G)
- Q1601 pad 2: /cell_S1_15/CELL+ -> CELL_1_POSITIVE
- Q1601 pad 3: Net-(Q1601-G) -> /cell_S1_15/CELL+
- Q201 pad 1: /cell_S1_1/CELL+ -> Net-(Q201-G)
- Q201 pad 2: /cell_S1_1/CELL+ -> PACK_+
- Q201 pad 3: Net-(Q201-G) -> /cell_S1_1/CELL+
- Q301 pad 1: /cell_S1_2/CELL+ -> Net-(Q301-G)
- Q301 pad 2: /cell_S1_2/CELL+ -> PACK_+
- Q301 pad 3: Net-(Q301-G) -> /cell_S1_2/CELL+
- Q401 pad 1: /cell_S1_3/CELL+ -> Net-(Q401-G)
- Q401 pad 2: /cell_S1_3/CELL+ -> PACK_+
- Q401 pad 3: Net-(Q401-G) -> /cell_S1_3/CELL+
- Q501 pad 1: /cell_S1_4/CELL+ -> Net-(Q501-G)
- Q501 pad 2: /cell_S1_4/CELL+ -> PACK_+
- Q501 pad 3: Net-(Q501-G) -> /cell_S1_4/CELL+
- Q601 pad 1: /cell_S1_5/CELL+ -> Net-(Q601-G)
- Q601 pad 2: /cell_S1_5/CELL+ -> PACK_+
- Q601 pad 3: Net-(Q601-G) -> /cell_S1_5/CELL+
- Q701 pad 1: /cell_S1_6/CELL+ -> Net-(Q701-G)
- Q701 pad 2: /cell_S1_6/CELL+ -> CELL_2_POSITIVE
- Q701 pad 3: Net-(Q701-G) -> /cell_S1_6/CELL+
- Q801 pad 1: /cell_S1_7/CELL+ -> Net-(Q801-G)
- Q801 pad 2: /cell_S1_7/CELL+ -> CELL_2_POSITIVE
- Q801 pad 3: Net-(Q801-G) -> /cell_S1_7/CELL+
- Q901 pad 1: /cell_S1_8/CELL+ -> Net-(Q901-G)
- Q901 pad 2: /cell_S1_8/CELL+ -> CELL_2_POSITIVE
- Q901 pad 3: Net-(Q901-G) -> /cell_S1_8/CELL+

Commit message: Solar battery WIP
Parts:
- removed BUZZER1901: MLT-7525, cacophony-library:BUZ-SMD_4P-L7.5-W7.5-P7.59-TL
- removed the C1702 at (77.6, -24.1)
- removed the C1703 at (77.6, -18.9)
- removed the C1901 at (131.2, -2.16)
- removed the D1701 at (77.1, -22.5)
- removed D1702: D, Diode_SMD:D_SOD-323_HandSoldering
- removed D1703: D_Shockley, Diode_SMD:D_SOD-523
- removed J1701: Conn_01x02, Connector_PinHeader_2.54mm:PinHeader_1x02_P2.54mm_Vertical
- removed Q1701, Q1702: CSD17578Q3A, Package_SON:VSON-8_3.3x3.3mm_P0.65mm_NexFET
- removed the R1702 at (70.9, 5.50)
- removed the R1703 at (70.9, 6.60)
- removed the TP1903 at (74.4, 11.4)
- removed the TP1904 at (76.0, 11.4)
- removed TP1908: TestPoint, cacophony-library:TP_PAD
- removed the U1701 at (82.0, -21.5)
- added BUZZER1902: PS1240P02CT3, cacophony-library:BUZ-TH_BD12.5-P5.00-D0.9, F.Cu at (78.5, -21.2)
- added C101: 1uF, Capacitor_SMD:C_0603_1608Metric, F.Cu at (66.4, -17.5)
- added C102: 1uF, Capacitor_SMD:C_0603_1608Metric, F.Cu at (66.4, -11.0)
- added C1708: 100uF 50V, Capacitor_THT:CP_Radial_D6.3mm_P2.50mm, B.Cu at (68.5, -27.8)
- added C1719: 100uF 50V, Capacitor_THT:CP_Radial_D6.3mm_P2.50mm, B.Cu at (69.8, 6.66)
- added D102: D, Diode_SMD:D_SOD-323_HandSoldering, F.Cu at (68.9, -12.3)
- added D103: D, Diode_SMD:D_SOD-323_HandSoldering, F.Cu at (68.9, -16.5)
- added D1901: D, Diode_SMD:D_SOD-323_HandSoldering, F.Cu at (86.3, -18.1)
- added JP101: Jumper_2_Open, Connector_PinHeader_2.00mm:PinHeader_2x01_P2.00mm_Vertical, B.Cu at (64.4, 12.5)
- added JP102: SolderJumper_2_Bridged, cacophony-library:SolderJumper-2_P1.3mm_Bridged_RoundedPad1.0x1.5mm, F.Cu at (65.0, 10.0)
- added Q102: 2N7002, Package_TO_SOT_SMD:SOT-23, F.Cu at (84.3, 6.24)
- added Q1901: 2N7002, Package_TO_SOT_SMD:SOT-23, F.Cu at (89.9, -16.8)
- added R103: 30k, Resistor_SMD:R_0402_1005Metric, F.Cu at (85.8, 4.68)
- added R104: 10k, Resistor_SMD:R_0402_1005Metric, F.Cu at (85.8, 2.80)
- added R1901: 10k, Resistor_SMD:R_0402_1005Metric, F.Cu at (77.8, 13.9)
- added R1902: 10k, Resistor_SMD:R_0402_1005Metric, F.Cu at (77.8, 14.9)
- added R1904: 0Ω, Resistor_SMD:R_0805_2012Metric, F.Cu at (89.2, -19.5)
- added TP1906: TestPoint, cacophony-library:TP_PAD, F.Cu at (84.8, -12.5)
- added TP1907: TestPoint, cacophony-library:TP_PAD, F.Cu at (87.2, -13.5)
- added U101: HT75xx-1-SOT89, Package_TO_SOT_SMD:SOT-89-3, F.Cu at (65.7, -14.3)
- BAT_N101, BAT_N102, BAT_N103, BAT_N104, BAT_N105, BAT_N106, BAT_N107, BAT_N108, BAT_N109, BAT_N110, BAT_N111, BAT_N112, BAT_N113, BAT_N114, BAT_N115: footprint cacophony-library:BAT-TH_MY-18650-05-J -> cacophony-library:BAT-TH_MY-18650-05-J-2
- BAT_P101, BAT_P102, BAT_P103, BAT_P104, BAT_P105, BAT_P106, BAT_P107, BAT_P108, BAT_P109, BAT_P110, BAT_P111, BAT_P112, BAT_P113, BAT_P114, BAT_P115: footprint cacophony-library:BAT-TH_MY-18650-04-J -> cacophony-library:BAT-TH_MY-18650-test8_4.0_2.5
- J1901: value Conn_01x04 -> TC2030; footprint Connector_PinHeader_2.00mm:PinHeader_1x04_P2.00mm_Vertical -> Connector:Tag-Connect_TC2030-IDC-NL_2x03_P1.27mm_Vertical; moved to B.Cu
- L1701: footprint cacophony-library:IND-SMD_L11.3-W10.0_XAL1010-332ME -> Inductor_SMD:L_TDK_SLF10165
- R1002, R1102, R1202, R1302, R1402, R1502, R1602, R202, R302, R402, R502, R602, R702, R802, R902: value 100k -> 330Ω
- R1003, R1103, R1203, R1303, R1403, R1503, R1603, R203, R303, R403, R503, R603, R703, R803, R903: value 330Ω -> 100k
- R1004, R1104, R1204, R1304, R1404, R1504, R1604, R204, R304, R404, R504, R604, R704, R804, R904: value 22mΩ -> 4.7M; footprint Resistor_SMD:R_0805_2012Metric -> Resistor_SMD:R_0402_1005Metric
- R1006, R1106, R1206, R1306, R1406, R1506, R1606, R206, R306, R406, R506, R606, R706, R806, R906: value 4.7M -> 2.2k
- R1007, R1107, R1207, R1307, R1407, R1507, R1607, R207, R307, R407, R507, R607, R707, R807, R907: value 2.2k -> 22mΩ; footprint Resistor_SMD:R_0402_1005Metric -> Resistor_SMD:R_0805_2012Metric
- U1801: footprint cacophony-library:TSSOP-20_4.4x6.5mm_P0.65mm -> Package_SO:TSSOP-20_4.4x6.5mm_P0.65mm
- moved Q301 201.6 mm to (-70.3, -30.8), turned to 90 degrees
- moved Q201 190.1 mm to (-74.4, -30.8), turned to 90 degrees
- moved Q501 186.9 mm to (-51.0, -30.8), turned to 90 degrees
- moved Q401 181.5 mm to (-55.1, -30.8), turned to 90 degrees
- moved Q601 170.9 mm to (-35.8, -30.8), turned to 90 degrees
- moved Q701 155.5 mm to (-31.7, 30.8), turned to -90 degrees
- moved Q801 138.9 mm to (-16.5, 30.8), turned to -90 degrees
- moved Q901 121.8 mm to (-12.4, 30.8), turned to -90 degrees
- moved Q1201 118.1 mm to (22.1, -30.8), turned to 90 degrees
- moved Q1101 112.4 mm to (6.88, 30.8), turned to -90 degrees
- moved Q1301 109.6 mm to (26.2, -30.8), turned to 90 degrees
- moved Q1001 108.0 mm to (2.77, 30.8), turned to -90 degrees
- moved Q1401 104.6 mm to (41.4, -30.8), turned to 90 degrees
- moved Q1601 100.2 mm to (60.7, -30.8), turned to 90 degrees
- moved Q1501 97.0 mm to (45.5, -30.8), turned to 90 degrees
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- renumbered C1716 to C1701, C1719 to C1702, C1720 to C1703, C1722 to C1704, C1704 to C1705, C1705 to C1706, C1706 to C1707, C1701 to C1709, C1709 to C1710, C1712 to C1711, C1713 to C1712, C1714 to C1713, C1715 to C1714, C1717 to C1715, C1721 to C1716, C1723 to C1717, C1707 to C1718, C1718 to C1720, C1708 to C1721, C1710 to C1722, C1711 to C1723, C1803 to C1801, C1810 to C1802, C1804 to C1803, C1805 to C1804, C1806 to C1805, C1813 to C1806, C1812 to C1807, C1807 to C1808, C1811 to C1809, C1801 to C1810, C1802 to C1811, C1808 to C1812, C1809 to C1813, C1903 to C1901, D1704 to D1701, D1901 to D1902, F102 to F101, F101 to F102, FL102 to FL101, FL101 to FL102, H113 to H102, H125 to H103, H109 to H104, H102 to H105, H114 to H106, H126 to H107, H110 to H108, H103 to H109, H115 to H110, H127 to H111, H111 to H112, H104 to H113, H116 to H114, H128 to H115, H121 to H116, H105 to H117, H117 to H118, H129 to H119, H122 to H120, H106 to H121, H118 to H122, H130 to H123, H123 to H124, H107 to H125, H119 to H126, H131 to H127, H112 to H128, H108 to H129, H120 to H130, H132 to H131, H124 to H132, J103 to J101, J101 to J102, J102 to J103, Q1802 to Q1801, Q1801 to Q1802, R1705 to R1701, R1707 to R1702, R1701 to R1703, R1708 to R1704, R1710 to R1705, R1704 to R1707, R1709 to R1708, R1811 to R1801, R1801 to R1802, R1802 to R1803, R1803 to R1804, R1804 to R1805, R1814 to R1806, R1805 to R1807, R1806 to R1808, R1812 to R1809, R1807 to R1810, R1809 to R1811, R1810 to R1812, R1808 to R1814, R1902 to R1903, R1903 to R1905, R1901 to R1906, TP1906 to TP1901, TP1907 to TP1902, TP1901 to TP1903, TP1902 to TP1904, U1702 to U1701, U1902 to U1901, U1901 to U1902
Connections:
- net /ATtiny1616/AHT21_VDD renamed /ATtiny1616/AHT20_VDD
- net /cell_S1_1/CELL+ renamed /cell_01/CELL+
- net /cell_S1_15/CELL+ renamed /cell_15/CELL+
- net /cell_S1_8/CELL+ renamed /cell_08/CELL+
- net Net-(D1704-A) renamed /BQ25798/STAT
- net Net-(D1704-K) renamed /BQ25798/STAT_PHY
- net Net-(D1901-A) renamed /ATtiny1616/LED
- net Net-(U1702-BATP) renamed /BQ25798/BATP
- net Net-(U1702-TS) renamed /BQ25798/TS
- net Net-(U1902-PB5) renamed /ATtiny1616/LED_PHY
- BAT_N101 pad 1: /cell_S1_1/CELL- -> /cell_01/CELL-
- BAT_N102 pad 1: /cell_S1_6/CELL- -> /cell_02/CELL-
- BAT_N103 pad 1: /cell_S1_11/CELL- -> /cell_03/CELL-
- BAT_N104 pad 1: /cell_S1_2/CELL- -> /cell_04/CELL-
- BAT_N105 pad 1: /cell_S1_7/CELL- -> /cell_05/CELL-
- BAT_N106 pad 1: /cell_S1_12/CELL- -> /cell_06/CELL-
- BAT_N107 pad 1: /cell_S1_3/CELL- -> /cell_07/CELL-
- BAT_N108 pad 1: /cell_S1_8/CELL- -> /cell_08/CELL-
- BAT_N109 pad 1: /cell_S1_13/CELL- -> /cell_09/CELL-
- BAT_N110 pad 1: /cell_S1_4/CELL- -> /cell_10/CELL-
- BAT_N111 pad 1: /cell_S1_9/CELL- -> /cell_11/CELL-
- BAT_N112 pad 1: /cell_S1_14/CELL- -> /cell_12/CELL-
- BAT_N113 pad 1: /cell_S1_5/CELL- -> /cell_13/CELL-
- BAT_N114 pad 1: /cell_S1_10/CELL- -> /cell_14/CELL-
- BAT_N115 pad 1: /cell_S1_15/CELL- -> /cell_15/CELL-
- BAT_P102 pad 1: /cell_S1_6/CELL+ -> /cell_02/CELL+
- BAT_P103 pad 1: /cell_S1_11/CELL+ -> /cell_03/CELL+
- BAT_P104 pad 1: /cell_S1_2/CELL+ -> /cell_04/CELL+
- BAT_P105 pad 1: /cell_S1_7/CELL+ -> /cell_05/CELL+
- BAT_P106 pad 1: /cell_S1_12/CELL+ -> /cell_06/CELL+
- BAT_P107 pad 1: /cell_S1_3/CELL+ -> /cell_07/CELL+
- BAT_P109 pad 1: /cell_S1_13/CELL+ -> /cell_09/CELL+
- BAT_P110 pad 1: /cell_S1_4/CELL+ -> /cell_10/CELL+
- BAT_P111 pad 1: /cell_S1_9/CELL+ -> /cell_11/CELL+
- BAT_P112 pad 1: /cell_S1_14/CELL+ -> /cell_12/CELL+
- BAT_P113 pad 1: /cell_S1_5/CELL+ -> /cell_13/CELL+
- BAT_P114 pad 1: /cell_S1_10/CELL+ -> /cell_14/CELL+
- C1001 pad 2: /cell_S1_9/CELL- -> /cell_09/CELL-
- C1101 pad 2: /cell_S1_10/CELL- -> /cell_10/CELL-
- C1201 pad 2: /cell_S1_11/CELL- -> /cell_11/CELL-
- C1301 pad 2: /cell_S1_12/CELL- -> /cell_12/CELL-
- C1401 pad 2: /cell_S1_13/CELL- -> /cell_13/CELL-
- C1501 pad 2: /cell_S1_14/CELL- -> /cell_14/CELL-
- C1601 pad 2: /cell_S1_15/CELL- -> /cell_15/CELL-
- C1705 pad 1: /BQ25798/VBUS -> V_{IN}
- C1706 pad 1: /BQ25798/VBUS -> V_{IN}
- C1707 pad 1: /BQ25798/VBUS -> V_{IN}
- C1716 pad 1: Net-(J1701-Pin_1) -> PACK_+
- C1717 pad 1: Net-(J1701-Pin_1) -> PACK_+
- C201 pad 2: /cell_S1_1/CELL- -> /cell_01/CELL-
- C301 pad 2: /cell_S1_2/CELL- -> /cell_02/CELL-
- C401 pad 2: /cell_S1_3/CELL- -> /cell_03/CELL-
- C501 pad 2: /cell_S1_4/CELL- -> /cell_04/CELL-
- C601 pad 2: /cell_S1_5/CELL- -> /cell_05/CELL-
- C701 pad 2: /cell_S1_6/CELL- -> /cell_06/CELL-
- C801 pad 2: /cell_S1_7/CELL- -> /cell_07/CELL-
- C901 pad 2: /cell_S1_8/CELL- -> /cell_08/CELL-
- FL102 pad 1: /GND_IN_PHY -> /POWER_IN_FUSED
- FL102 pad 2: /POWER_IN_FUSED -> /GND_IN_PHY
- FL102 pad 3: /POWER_IN_FILTERED -> GND
- FL102 pad 4: GND -> /POWER_IN_FILTERED
- J1901 pad 1: /ATtiny1616/UPDI -> RX
- J1901 pad 2: GND -> Net-(J1901-Pad2)
- J1901 pad 3: RX -> TX
- J1901 pad 4: TX -> Net-(J1901-Pad4)
- Q1001 pad 3: /cell_S1_9/CELL+ -> /cell_09/CELL+
- Q1002 pad 1: /cell_S1_9/CELL+ -> /cell_09/CELL+
- Q1003 pad 1: /cell_S1_9/BAT_NEG -> /cell_09/BAT_NEG
- Q1101 pad 3: /cell_S1_10/CELL+ -> /cell_10/CELL+
- Q1102 pad 1: /cell_S1_10/CELL+ -> /cell_10/CELL+
- Q1103 pad 1: /cell_S1_10/BAT_NEG -> /cell_10/BAT_NEG
- Q1201 pad 3: /cell_S1_11/CELL+ -> /cell_11/CELL+
- Q1202 pad 1: /cell_S1_11/CELL+ -> /cell_11/CELL+
- Q1203 pad 1: /cell_S1_11/BAT_NEG -> /cell_11/BAT_NEG
- Q1301 pad 3: /cell_S1_12/CELL+ -> /cell_12/CELL+
- Q1302 pad 1: /cell_S1_12/CELL+ -> /cell_12/CELL+
- Q1303 pad 1: /cell_S1_12/BAT_NEG -> /cell_12/BAT_NEG
- Q1401 pad 3: /cell_S1_13/CELL+ -> /cell_13/CELL+
- Q1402 pad 1: /cell_S1_13/CELL+ -> /cell_13/CELL+
- Q1403 pad 1: /cell_S1_13/BAT_NEG -> /cell_13/BAT_NEG
- Q1501 pad 3: /cell_S1_14/CELL+ -> /cell_14/CELL+
- Q1502 pad 1: /cell_S1_14/CELL+ -> /cell_14/CELL+
- Q1503 pad 1: /cell_S1_14/BAT_NEG -> /cell_14/BAT_NEG
- Q1603 pad 1: /cell_S1_15/BAT_NEG -> /cell_15/BAT_NEG
- Q201 pad 2: PACK_+ -> /PACK_+_PHY
- Q202 pad 2: PACK_+ -> /PACK_+_PHY
- Q203 pad 1: /cell_S1_1/BAT_NEG -> /cell_01/BAT_NEG
- Q301 pad 2: PACK_+ -> /PACK_+_PHY
- Q301 pad 3: /cell_S1_2/CELL+ -> /cell_02/CELL+
- Q302 pad 1: /cell_S1_2/CELL+ -> /cell_02/CELL+
- Q302 pad 2: PACK_+ -> /PACK_+_PHY
- Q303 pad 1: /cell_S1_2/BAT_NEG -> /cell_02/BAT_NEG
- Q401 pad 2: PACK_+ -> /PACK_+_PHY
- Q401 pad 3: /cell_S1_3/CELL+ -> /cell_03/CELL+
- Q402 pad 1: /cell_S1_3/CELL+ -> /cell_03/CELL+
- Q402 pad 2: PACK_+ -> /PACK_+_PHY
- Q403 pad 1: /cell_S1_3/BAT_NEG -> /cell_03/BAT_NEG
- Q501 pad 2: PACK_+ -> /PACK_+_PHY
- Q501 pad 3: /cell_S1_4/CELL+ -> /cell_04/CELL+
- Q502 pad 1: /cell_S1_4/CELL+ -> /cell_04/CELL+
- Q502 pad 2: PACK_+ -> /PACK_+_PHY
- Q503 pad 1: /cell_S1_4/BAT_NEG -> /cell_04/BAT_NEG
- Q601 pad 2: PACK_+ -> /PACK_+_PHY
- Q601 pad 3: /cell_S1_5/CELL+ -> /cell_05/CELL+
- Q602 pad 1: /cell_S1_5/CELL+ -> /cell_05/CELL+
- Q602 pad 2: PACK_+ -> /PACK_+_PHY
- Q603 pad 1: /cell_S1_5/BAT_NEG -> /cell_05/BAT_NEG
- Q701 pad 3: /cell_S1_6/CELL+ -> /cell_06/CELL+
- Q702 pad 1: /cell_S1_6/CELL+ -> /cell_06/CELL+
- Q703 pad 1: /cell_S1_6/BAT_NEG -> /cell_06/BAT_NEG
- Q801 pad 3: /cell_S1_7/CELL+ -> /cell_07/CELL+
- Q802 pad 1: /cell_S1_7/CELL+ -> /cell_07/CELL+
- Q803 pad 1: /cell_S1_7/BAT_NEG -> /cell_07/BAT_NEG
- Q903 pad 1: /cell_S1_8/BAT_NEG -> /cell_08/BAT_NEG
- R1001 pad 1: /cell_S1_9/CELL+ -> /cell_09/CELL+
- R1002 pad 1: /cell_S1_9/CELL- -> CELL_2_POSITIVE
- R1002 pad 2: Net-(Q1001-G) -> Net-(U1001-BAT)
- R1003 pad 1: CELL_2_POSITIVE -> /cell_09/CELL-
- R1003 pad 2: Net-(U1001-BAT) -> Net-(Q1001-G)
- R1004 pad 1: /cell_S1_9/CELL- -> Net-(Q1003-G1)
- R1004 pad 2: /cell_S1_9/BAT_NEG -> /cell_09/BAT_NEG
- R1005 pad 1: Net-(Q1003-G1) -> Net-(Q1003-G2)
- R1005 pad 2: /cell_S1_9/BAT_NEG -> CELL_1_POSITIVE
- R1006 pad 1: Net-(Q1003-G2) -> Net-(U1001-V-)
- R1007 pad 1: Net-(U1001-V-) -> /cell_09/CELL-
- R1007 pad 2: CELL_1_POSITIVE -> /cell_09/BAT_NEG
- R1101 pad 1: /cell_S1_10/CELL+ -> /cell_10/CELL+
- R1102 pad 1: /cell_S1_10/CELL- -> CELL_2_POSITIVE
- R1102 pad 2: Net-(Q1101-G) -> Net-(U1101-BAT)
- R1103 pad 1: CELL_2_POSITIVE -> /cell_10/CELL-
- R1103 pad 2: Net-(U1101-BAT) -> Net-(Q1101-G)
- R1104 pad 1: /cell_S1_10/CELL- -> Net-(Q1103-G1)
- R1104 pad 2: /cell_S1_10/BAT_NEG -> /cell_10/BAT_NEG
- R1105 pad 1: Net-(Q1103-G1) -> Net-(Q1103-G2)
- R1105 pad 2: /cell_S1_10/BAT_NEG -> CELL_1_POSITIVE
- R1106 pad 1: Net-(Q1103-G2) -> Net-(U1101-V-)
- R1107 pad 1: Net-(U1101-V-) -> /cell_10/CELL-
- R1107 pad 2: CELL_1_POSITIVE -> /cell_10/BAT_NEG
- R1201 pad 1: /cell_S1_11/CELL+ -> /cell_11/CELL+
- R1202 pad 1: /cell_S1_11/CELL- -> CELL_1_POSITIVE
- R1202 pad 2: Net-(Q1201-G) -> Net-(U1201-BAT)
- R1203 pad 1: CELL_1_POSITIVE -> /cell_11/CELL-
- R1203 pad 2: Net-(U1201-BAT) -> Net-(Q1201-G)
- R1204 pad 1: /cell_S1_11/CELL- -> Net-(Q1203-G1)
- R1204 pad 2: /cell_S1_11/BAT_NEG -> /cell_11/BAT_NEG
- R1205 pad 1: Net-(Q1203-G1) -> Net-(Q1203-G2)
- R1205 pad 2: /cell_S1_11/BAT_NEG -> GND
- R1206 pad 1: Net-(Q1203-G2) -> Net-(U1201-V-)
- R1207 pad 1: Net-(U1201-V-) -> /cell_11/CELL-
- R1207 pad 2: GND -> /cell_11/BAT_NEG
- R1301 pad 1: /cell_S1_12/CELL+ -> /cell_12/CELL+
- R1302 pad 1: /cell_S1_12/CELL- -> CELL_1_POSITIVE
- R1302 pad 2: Net-(Q1301-G) -> Net-(U1301-BAT)
- R1303 pad 1: CELL_1_POSITIVE -> /cell_12/CELL-
- R1303 pad 2: Net-(U1301-BAT) -> Net-(Q1301-G)
- R1304 pad 1: /cell_S1_12/CELL- -> Net-(Q1303-G1)
- R1304 pad 2: /cell_S1_12/BAT_NEG -> /cell_12/BAT_NEG
- R1305 pad 1: Net-(Q1303-G1) -> Net-(Q1303-G2)
- R1305 pad 2: /cell_S1_12/BAT_NEG -> GND
- R1306 pad 1: Net-(Q1303-G2) -> Net-(U1301-V-)
- R1307 pad 1: Net-(U1301-V-) -> /cell_12/CELL-
- R1307 pad 2: GND -> /cell_12/BAT_NEG
- R1401 pad 1: /cell_S1_13/CELL+ -> /cell_13/CELL+
- R1402 pad 1: /cell_S1_13/CELL- -> CELL_1_POSITIVE
- R1402 pad 2: Net-(Q1401-G) -> Net-(U1401-BAT)
- R1403 pad 1: CELL_1_POSITIVE -> /cell_13/CELL-
- R1403 pad 2: Net-(U1401-BAT) -> Net-(Q1401-G)
- R1404 pad 1: /cell_S1_13/CELL- -> Net-(Q1403-G1)
- R1404 pad 2: /cell_S1_13/BAT_NEG -> /cell_13/BAT_NEG
- R1405 pad 1: Net-(Q1403-G1) -> Net-(Q1403-G2)
- R1405 pad 2: /cell_S1_13/BAT_NEG -> GND
- R1406 pad 1: Net-(Q1403-G2) -> Net-(U1401-V-)
- R1407 pad 1: Net-(U1401-V-) -> /cell_13/CELL-
- R1407 pad 2: GND -> /cell_13/BAT_NEG
- R1501 pad 1: /cell_S1_14/CELL+ -> /cell_14/CELL+
- R1502 pad 1: /cell_S1_14/CELL- -> CELL_1_POSITIVE
- R1502 pad 2: Net-(Q1501-G) -> Net-(U1501-BAT)
- R1503 pad 1: CELL_1_POSITIVE -> /cell_14/CELL-
- R1503 pad 2: Net-(U1501-BAT) -> Net-(Q1501-G)
- R1504 pad 1: /cell_S1_14/CELL- -> Net-(Q1503-G1)
- R1504 pad 2: /cell_S1_14/BAT_NEG -> /cell_14/BAT_NEG
- R1505 pad 1: Net-(Q1503-G1) -> Net-(Q1503-G2)
- R1505 pad 2: /cell_S1_14/BAT_NEG -> GND
- R1506 pad 1: Net-(Q1503-G2) -> Net-(U1501-V-)
- R1507 pad 1: Net-(U1501-V-) -> /cell_14/CELL-
- R1507 pad 2: GND -> /cell_14/BAT_NEG
- R1602 pad 1: /cell_S1_15/CELL- -> CELL_1_POSITIVE
- R1602 pad 2: Net-(Q1601-G) -> Net-(U1601-BAT)
- R1603 pad 1: CELL_1_POSITIVE -> /cell_15/CELL-
- R1603 pad 2: Net-(U1601-BAT) -> Net-(Q1601-G)
- R1604 pad 1: /cell_S1_15/CELL- -> Net-(Q1603-G1)
- R1604 pad 2: /cell_S1_15/BAT_NEG -> /cell_15/BAT_NEG
- R1605 pad 1: Net-(Q1603-G1) -> Net-(Q1603-G2)
- R1605 pad 2: /cell_S1_15/BAT_NEG -> GND
- R1606 pad 1: Net-(Q1603-G2) -> Net-(U1601-V-)
- R1607 pad 1: Net-(U1601-V-) -> /cell_15/CELL-
- R1607 pad 2: GND -> /cell_15/BAT_NEG
- R1705 pad 2: Net-(J1701-Pin_1) -> PACK_+
- R1906 pad 1: +3V3 -> +3.3V
- R201 pad 2: PACK_+ -> /PACK_+_PHY
- R202 pad 1: /cell_S1_1/CELL- -> /PACK_+_PHY
- R202 pad 2: Net-(Q201-G) -> Net-(U201-BAT)
- R203 pad 1: PACK_+ -> /cell_01/CELL-
- R203 pad 2: Net-(U201-BAT) -> Net-(Q201-G)
- R204 pad 1: /cell_S1_1/CELL- -> Net-(Q203-G1)
- R204 pad 2: /cell_S1_1/BAT_NEG -> /cell_01/BAT_NEG
- R205 pad 1: Net-(Q203-G1) -> Net-(Q203-G2)
- R205 pad 2: /cell_S1_1/BAT_NEG -> CELL_2_POSITIVE
- R206 pad 1: Net-(Q203-G2) -> Net-(U201-V-)
- R207 pad 1: Net-(U201-V-) -> /cell_01/CELL-
- R207 pad 2: CELL_2_POSITIVE -> /cell_01/BAT_NEG
- R301 pad 1: /cell_S1_2/CELL+ -> /cell_02/CELL+
- R301 pad 2: PACK_+ -> /PACK_+_PHY
- R302 pad 1: /cell_S1_2/CELL- -> /PACK_+_PHY
- R302 pad 2: Net-(Q301-G) -> Net-(U301-BAT)
- R303 pad 1: PACK_+ -> /cell_02/CELL-
- R303 pad 2: Net-(U301-BAT) -> Net-(Q301-G)
- R304 pad 1: /cell_S1_2/CELL- -> Net-(Q303-G1)
- R304 pad 2: /cell_S1_2/BAT_NEG -> /cell_02/BAT_NEG
- R305 pad 1: Net-(Q303-G1) -> Net-(Q303-G2)
- R305 pad 2: /cell_S1_2/BAT_NEG -> CELL_2_POSITIVE
- R306 pad 1: Net-(Q303-G2) -> Net-(U301-V-)
- R307 pad 1: Net-(U301-V-) -> /cell_02/CELL-
- R307 pad 2: CELL_2_POSITIVE -> /cell_02/BAT_NEG
- R401 pad 1: /cell_S1_3/CELL+ -> /cell_03/CELL+
- R401 pad 2: PACK_+ -> /PACK_+_PHY
- R402 pad 1: /cell_S1_3/CELL- -> /PACK_+_PHY
- R402 pad 2: Net-(Q401-G) -> Net-(U401-BAT)
- R403 pad 1: PACK_+ -> /cell_03/CELL-
- R403 pad 2: Net-(U401-BAT) -> Net-(Q401-G)
- R404 pad 1: /cell_S1_3/CELL- -> Net-(Q403-G1)
- R404 pad 2: /cell_S1_3/BAT_NEG -> /cell_03/BAT_NEG
- R405 pad 1: Net-(Q403-G1) -> Net-(Q403-G2)
- R405 pad 2: /cell_S1_3/BAT_NEG -> CELL_2_POSITIVE
- R406 pad 1: Net-(Q403-G2) -> Net-(U401-V-)
- R407 pad 1: Net-(U401-V-) -> /cell_03/CELL-
- R407 pad 2: CELL_2_POSITIVE -> /cell_03/BAT_NEG
- R501 pad 1: /cell_S1_4/CELL+ -> /cell_04/CELL+
- R501 pad 2: PACK_+ -> /PACK_+_PHY
- R502 pad 1: /cell_S1_4/CELL- -> /PACK_+_PHY
- R502 pad 2: Net-(Q501-G) -> Net-(U501-BAT)
- R503 pad 1: PACK_+ -> /cell_04/CELL-
- R503 pad 2: Net-(U501-BAT) -> Net-(Q501-G)
- R504 pad 1: /cell_S1_4/CELL- -> Net-(Q503-G1)
- R504 pad 2: /cell_S1_4/BAT_NEG -> /cell_04/BAT_NEG
- R505 pad 1: Net-(Q503-G1) -> Net-(Q503-G2)
- R505 pad 2: /cell_S1_4/BAT_NEG -> CELL_2_POSITIVE
- R506 pad 1: Net-(Q503-G2) -> Net-(U501-V-)
- R507 pad 1: Net-(U501-V-) -> /cell_04/CELL-
- R507 pad 2: CELL_2_POSITIVE -> /cell_04/BAT_NEG
- R601 pad 1: /cell_S1_5/CELL+ -> /cell_05/CELL+
- R601 pad 2: PACK_+ -> /PACK_+_PHY
- R602 pad 1: /cell_S1_5/CELL- -> /PACK_+_PHY
- R602 pad 2: Net-(Q601-G) -> Net-(U601-BAT)
- R603 pad 1: PACK_+ -> /cell_05/CELL-
- R603 pad 2: Net-(U601-BAT) -> Net-(Q601-G)
- R604 pad 1: /cell_S1_5/CELL- -> Net-(Q603-G1)
- R604 pad 2: /cell_S1_5/BAT_NEG -> /cell_05/BAT_NEG
- R605 pad 1: Net-(Q603-G1) -> Net-(Q603-G2)
- R605 pad 2: /cell_S1_5/BAT_NEG -> CELL_2_POSITIVE
- R606 pad 1: Net-(Q603-G2) -> Net-(U601-V-)
- R607 pad 1: Net-(U601-V-) -> /cell_05/CELL-
- R607 pad 2: CELL_2_POSITIVE -> /cell_05/BAT_NEG
- R701 pad 1: /cell_S1_6/CELL+ -> /cell_06/CELL+
- R702 pad 1: /cell_S1_6/CELL- -> CELL_2_POSITIVE
- R702 pad 2: Net-(Q701-G) -> Net-(U701-BAT)
- R703 pad 1: CELL_2_POSITIVE -> /cell_06/CELL-
- R703 pad 2: Net-(U701-BAT) -> Net-(Q701-G)
- R704 pad 1: /cell_S1_6/CELL- -> Net-(Q703-G1)
- R704 pad 2: /cell_S1_6/BAT_NEG -> /cell_06/BAT_NEG
- R705 pad 1: Net-(Q703-G1) -> Net-(Q703-G2)
- R705 pad 2: /cell_S1_6/BAT_NEG -> CELL_1_POSITIVE
- R706 pad 1: Net-(Q703-G2) -> Net-(U701-V-)
- R707 pad 1: Net-(U701-V-) -> /cell_06/CELL-
- R707 pad 2: CELL_1_POSITIVE -> /cell_06/BAT_NEG
- R801 pad 1: /cell_S1_7/CELL+ -> /cell_07/CELL+
- R802 pad 1: /cell_S1_7/CELL- -> CELL_2_POSITIVE
- R802 pad 2: Net-(Q801-G) -> Net-(U801-BAT)
- R803 pad 1: CELL_2_POSITIVE -> /cell_07/CELL-
- R803 pad 2: Net-(U801-BAT) -> Net-(Q801-G)
- R804 pad 1: /cell_S1_7/CELL- -> Net-(Q803-G1)
- R804 pad 2: /cell_S1_7/BAT_NEG -> /cell_07/BAT_NEG
- R805 pad 1: Net-(Q803-G1) -> Net-(Q803-G2)
- R805 pad 2: /cell_S1_7/BAT_NEG -> CELL_1_POSITIVE
- R806 pad 1: Net-(Q803-G2) -> Net-(U801-V-)
- R807 pad 1: Net-(U801-V-) -> /cell_07/CELL-
- R807 pad 2: CELL_1_POSITIVE -> /cell_07/BAT_NEG
- R902 pad 1: /cell_S1_8/CELL- -> CELL_2_POSITIVE
- R902 pad 2: Net-(Q901-G) -> Net-(U901-BAT)
- R903 pad 1: CELL_2_POSITIVE -> /cell_08/CELL-
- R903 pad 2: Net-(U901-BAT) -> Net-(Q901-G)
- R904 pad 1: /cell_S1_8/CELL- -> Net-(Q903-G1)
- R904 pad 2: /cell_S1_8/BAT_NEG -> /cell_08/BAT_NEG
- R905 pad 1: Net-(Q903-G1) -> Net-(Q903-G2)
- R905 pad 2: /cell_S1_8/BAT_NEG -> CELL_1_POSITIVE
- R906 pad 1: Net-(Q903-G2) -> Net-(U901-V-)
- R907 pad 1: Net-(U901-V-) -> /cell_08/CELL-
- R907 pad 2: CELL_1_POSITIVE -> /cell_08/BAT_NEG
- TP1902 pad 1: Net-(U1902-PA2) -> Net-(U1901-PA4)
- U1001 pad 4: /cell_S1_9/CELL- -> /cell_09/CELL-
- U1101 pad 4: /cell_S1_10/CELL- -> /cell_10/CELL-
- U1201 pad 4: /cell_S1_11/CELL- -> /cell_11/CELL-
- U1301 pad 4: /cell_S1_12/CELL- -> /cell_12/CELL-
- U1401 pad 4: /cell_S1_13/CELL- -> /cell_13/CELL-
- U1501 pad 4: /cell_S1_14/CELL- -> /cell_14/CELL-
- U1601 pad 4: /cell_S1_15/CELL- -> /cell_15/CELL-
- U1701 pad 11: Net-(D1703-K) -> GND
- U1701 pad 2: /BQ25798/VBUS -> V_{IN}
- U1701 pad 22: Net-(J1701-Pin_1) -> PACK_+
- U1701 pad 23: Net-(J1701-Pin_1) -> PACK_+
- U1701 pad 3: /BQ25798/VBUS -> V_{IN}
- U1701 pad 6: /BQ25798/D+ -> unconnected-(U1701-D+-Pad6)
- U1701 pad 7: /BQ25798/D- -> unconnected-(U1701-D--Pad7)
- U1701 pad 8: /BQ25798/VBUS -> V_{IN}
- U1901 pad 1: Net-(U1902-PA2) -> ~{INT}
- U1901 pad 17: Net-(U1902-PC2) -> SENSE_DIV
- U1901 pad 18: Net-(U1902-PC3) -> PULL_SENSE_LOW
- U1901 pad 2: Net-(U1902-PA3) -> BUZZER
- U1901 pad 5: ~{INT} -> Net-(U1901-PA4)
- U201 pad 4: /cell_S1_1/CELL- -> /cell_01/CELL-
- U301 pad 4: /cell_S1_2/CELL- -> /cell_02/CELL-
- U401 pad 4: /cell_S1_3/CELL- -> /cell_03/CELL-
- U501 pad 4: /cell_S1_4/CELL- -> /cell_04/CELL-
- U601 pad 4: /cell_S1_5/CELL- -> /cell_05/CELL-
- U701 pad 4: /cell_S1_6/CELL- -> /cell_06/CELL-
- U801 pad 4: /cell_S1_7/CELL- -> /cell_07/CELL-
- U901 pad 4: /cell_S1_8/CELL- -> /cell_08/CELL-
Routing:
- net PACK_+: track 378.8 -> 69.0 mm, vias 26 -> 40
- net CELL_2_POSITIVE: track 365.9 -> 142.9 mm, vias 37 -> 32
- net CELL_1_POSITIVE: track 299.7 -> 127.7 mm, vias 37 -> 30
- net /cell_S1_6/CELL-: track 69.6 -> 0.00 mm
- net /cell_S1_8/CELL-: track 69.3 -> 0.00 mm
- net /cell_S1_10/CELL-: track 69.2 -> 0.00 mm
- net /cell_S1_4/CELL-: track 67.5 -> 0.00 mm
- net /cell_S1_14/CELL-: track 67.3 -> 0.00 mm
- net /cell_S1_12/CELL-: track 67.3 -> 0.00 mm
- net /cell_S1_2/CELL-: track 67.1 -> 0.00 mm
- net /cell_S1_9/CELL-: track 63.5 -> 0.00 mm
- net /cell_S1_7/CELL-: track 63.5 -> 0.00 mm
- net /cell_S1_11/CELL-: track 62.7 -> 0.00 mm
- net /cell_S1_3/CELL-: track 62.7 -> 0.00 mm
- net /cell_S1_13/CELL-: track 62.7 -> 0.00 mm
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- added copper zone on F.Cu, net /PACK_+_PHY
- added copper zone on In2.Cu, net /PACK_+_PHY
- added copper zone on F.Cu, net PACK_-
- added copper zone on F.Cu, net V_{IN}
- removed copper zone on F.Cu, net /BQ25798/VBUS
- removed copper zone on F.Cu, net CELL_1_POSITIVE
- removed copper zone on F.Cu, net CELL_2_POSITIVE
- removed copper zone on In2.Cu, net GND
- removed copper zone on F.Cu, net Net-(J1701-Pin_1)
Other:
- board size 175 x 85 mm -> 177 x 85 mm
- board text removed: "RX"
- board text removed: "TX"
- board text removed: "UPDI"

Commit message: Version v0.0.2
Routing:
- added copper zone on In2.Cu, net GND

Commit message: Tidy up of files
Other:
- outline, holes or cut-outs redrawn
