File: solar-BQ25798/BQ76920.kicad_sch (KiCad schematic)
At the start: 33 parts, among them Q1801 CSD17578Q3A, Q1802 Q_PMOS_GSD, Q1803 CSD17578Q3A, U1801 BQ76920PW

Commit message: Getting ready for v0.3.0
Connections:
- net CELL_3_POSITIVE is gone; now on net PACK_+: R1801.1
Other:
- note added: "BQ76200PWR"
