File: solar-BQ25798/BQ76920.kicad_sch (KiCad schematic)
At the start: 33 parts, among them Q1801 CSD17578Q3A, Q1802 Q_PMOS_GSD, Q1803 CSD17578Q3A, U1801 BQ76920PW

Commit message: Update LCSC part numbers
Parts:
- R1808: LCSC Part C875667 -> C875618
Changed lines of the file:
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@@
 			)
 		)
-		(property "LCSC Part" "C875667"
+		(property "LCSC Part" "C875618"
 			(at 130.81 146.05 90)
 			(hide yes)
