File: solar-BQ25798/solar-BQ25798.kicad_sch (KiCad schematic)
At the start: 88 parts, among them J101 Power In, J102 Power OUT, J103 Power OUT, Q1 Q_NMOS_GSD, Q101 DMP4013LFGQ-13, Q102 2N7002, U101 HT75xx-1-SOT89, U102 INA219AxDCN

Commit message: Getting ready for v0.3.0
Parts:
- removed C103: 100nF, Capacitor_SMD:C_0402_1005Metric, symbol Device:C_Small
- removed R103, R104: 100k, Resistor_SMD:R_0402_1005Metric, symbol Device:R
- removed R107: 0Ω, cacophony-library:R_1206_Shunt_Short, symbol cacophony-library:R_Shunt_Short
- removed U102: INA219AxDCN, Package_TO_SOT_SMD:SOT-23-8, symbol Sensor_Energy:INA219AxDCN
- added D1, D2, D3: SMAJ20CA, Diode_SMD:D_SMA, symbol Diode:SMAJ20CA
Connections:
- net GND_IN_PHY: now also D1.1 (A1)
- net GND_OUT_FILTERED: now also D2.2 (A2), D3.2 (A2)
- net POWER_IN_FUSED: now also D1.2 (A2)
- net V_BAT_FILTERED: now also D2.1 (A1)
- net V_{SENSE}: now also D3.1 (A1)
Other:
- note added: "SMAJxxA"
- moved on the sheet: D103, F101, F102, FL101, FL102, J101, J102, J103, Q101, Q102, R101, R102
