File: solar-BQ25798/solar-BQ25798.kicad_sch (KiCad schematic)
At the start: 86 parts, among them J101 Power In, J102 Power OUT, J103 Power OUT, Q1 Q_NMOS_GSD, Q101 DMP4013LFGQ-13, Q102 2N7002, U101 HT75xx-1-SOT89

Commit message: Change p-mosfet and fuse LCSC part number
Parts:
- F101, F102: LCSC Part C5220740 -> C136386
Changed lines of the file:
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@@
 			)
 		)
-		(property "LCSC Part" "C5220740"
+		(property "LCSC Part" "C136386"
 			(at 33.02 30.48 90)
 			(hide yes)
@@
 			)
 		)
-		(property "LCSC Part" "C5220740"
+		(property "LCSC Part" "C136386"
 			(at 265.43 25.4 90)
 			(hide yes)
