File: solar-BQ25798/attiny1616.kicad_sch (KiCad schematic)
At the start: 28 parts, among them J1901 TC2030, Q1901 2N7002, U106 M24C02-WMN, U1901 AHT20_C2757850, U1902 ATtiny1616-M

Commit message: Getting ready for v0.3.0
Parts:
- removed C1814, C1815: 4.7uF, Capacitor_SMD:C_0402_1005Metric, symbol Device:C_Small
- removed D1902: LED, LED_SMD:LED_0603_1608Metric, symbol Device:LED
- removed R1901: 330Ω, Resistor_SMD:R_0402_1005Metric, symbol Device:R
- removed R1904: 2.2k, Resistor_SMD:R_0402_1005Metric, symbol Device:R
- removed R1905, R1906: 10k, Resistor_SMD:R_0402_1005Metric, symbol Device:R
- removed U1901: AHT20_C2757850, cacophony-library:SENSOR-SMD_L3.0-W3.0-P1.00-BR, symbol cacophony-library:AHT20_C2757850
- added C122: 100nF, Capacitor_SMD:C_0402_1005Metric, symbol Device:C_Small
- added R1, R6: 4.7k, Resistor_SMD:R_0603_1608Metric, symbol Device:R
- added TP1904, TP1906: TestPoint, cacophony-library:TP_PAD_S, symbol cacophony-library:TestPoint
- added U1: HDC2080, Sensor_Humidity:Texas_S-PWSON-N6-HDC2080, symbol Sensor_Humidity:HDC2080
- TP1902, TP1903, TP1905, TP1908, TP1909: footprint cacophony-library:TP_PAD -> cacophony-library:TP_PAD_S
Connections:
- net +3.3V: now also C122.2, R1.2, R6.2, U1.5 (VDD)
- net GND: now also C122.1, U1.2 (GND), U1.3 (ADDR)
- net SCL: now also R6.1, U1.6 (SCL)
- net SDA: now also R1.1, U1.1 (SDA)
- net LED_PHY: no longer names the net of U1902.9 (PB5)
- net LED_PHY: now also TP1906.1
- new net: TP1904.1, U1.4 (DRDY)
- no-connect marks 5 -> 3
Other:
- note added: "I2C Address 0x40"
- note removed: "I2C Address 0x38"

Commit message: Tidy up
Connections:
- net BUZZER_DRAIN: now reaches Q1901.3 (D), R1902.1 (A)
- net BUZZER_N: now reaches BUZZER1.2, R1902.2 (B), R2.2, R3.2, R4.2
- net PB4: now reaches TP1903.1, U1902.10 (PB4)
- net T_SW_SENSE_PIN: now reaches R1908.1, U1902.20 (PA1)
- net UPDI_PIN: now reaches R1903.1, U1902.19 (~{RESET}/PA0)
- net PA4: now reaches TP1905.1, U1902.5 (PA4)
- net PC2: now reaches TP1908.1, U1902.17 (PC2)
- net PC3: now reaches TP1902.1, U1902.18 (PC3)
- net PB5: now reaches TP1906.1, U1902.9 (PB5)
Other:
- moved on the sheet: J1901, Q1901, R1902, R1903, TP1902, TP1903, TP1905, TP1906, TP1908, TP1909
