File: solar-BQ25798/cell.kicad_sch (KiCad schematic)
At the start: 12 parts, among them Q201 DMP2035U-7, Q202 Q_PMOS_GSD, Q203 FS8205A_C908265, U201 BQ297xy

Commit message: Tidy up
Connections:
- net RP_GATE: now reaches Q201.1 (G), Q202.3 (D), R202.2
- net C_{OUT}: now reaches Q203.4 (G2), R206.1, U201.2 (Cout)
- net V-: now reaches R207.1, U201.6 (V-)
- net D_{OUT}: now reaches Q203.6 (G1), R205.1, U201.3 (Dout)
- net BAT: now reaches C201.1, R203.2, U201.5 (BAT)
Other:
- moved on the sheet: C201
Changed lines of the file:
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@@
 	(wire
 		(pts
-			(xy 148.59 92.71) (xy 148.59 93.98)
+			(xy 148.59 92.71) (xy 148.59 99.06)
 		)
 		(stroke
@@
 	(wire
 		(pts
-			(xy 148.59 99.06) (xy 148.59 132.08)
+			(xy 148.59 104.14) (xy 148.59 132.08)
 		)
 		(stroke
@@
 		)
 	)
+	(label "BAT"
+		(at 152.4 92.71 0)
+		(effects
+			(font
+				(size 1.27 1.27)
+			)
+			(justify left bottom)
+		)
+	)
+	(label "C_{OUT}"
+		(at 190.5 92.71 0)
+		(effects
+			(font
+				(size 1.27 1.27)
+			)
+			(justify left bottom)
+		)
+	)
+	(label "V-"
+		(at 163.83 81.28 0)
+		(effects
+			(font
+				(size 1.27 1.27)
+			)
+			(justify left bottom)
+		)
+	)
 	(label "BAT_NEG"
 		(at 182.88 132.08 0)
+		(effects
+			(font
+				(size 1.27 1.27)
+			)
+			(justify left bottom)
+		)
+	)
+	(label "RP_GATE"
+		(at 106.68 96.52 0)
+		(effects
+			(font
+				(size 1.27 1.27)
+			)
+			(justify left bottom)
+		)
+	)
+	(label "D_{OUT}"
+		(at 189.23 97.79 0)
 		(effects
 			(font
@@
 	(symbol
 		(lib_id "Device:C_Small")
-		(at 148.59 96.52 0)
+		(at 148.59 101.6 0)
 		(unit 1)
 		(body_style 1)
@@
 		(fields_autoplaced yes)
 		(property "Reference" "C201"
-			(at 151.13 95.2562 0)
+			(at 151.13 100.3362 0)
 			(show_name no)
 			(do_not_autoplace no)
@@
 		)
 		(property "Value" "100nF"
-			(at 151.13 97.7962 0)
+			(at 151.13 102.8762 0)
 			(show_name no)
 			(do_not_autoplace no)
@@
 		)
 		(property "Footprint" "Capacitor_SMD:C_0402_1005Metric"
-			(at 148.59 96.52 0)
+			(at 148.59 101.6 0)
 			(hide yes)
 			(show_name no)
@@
 		)
 		(property "Datasheet" ""
-			(at 148.59 96.52 0)
+			(at 148.59 101.6 0)
 			(hide yes)
 			(show_name no)
@@
 		)
 		(property "Description" "Unpolarized capacitor, small symbol"
-			(at 148.59 96.52 0)
+			(at 148.59 101.6 0)
 			(hide yes)
 			(show_name no)
@@
 		)
 		(property "LCSC Part" "C1525"
-			(at 148.59 96.52 0)
+			(at 148.59 101.6 0)
 			(hide yes)
 			(show_name no)
@@
 		)
 		(property "JLCPCB" ""
-			(at 148.59 96.52 0)
-			(hide yes)
-			(show_name no)
+			(at 148.59 101.6 0)
+			(hide yes)
+			(show_name no)
