File: solar-programmer/solar-programmer/solar-programmer.kicad_sch (KiCad schematic)
At the start: 22 parts, among them J1 Raspberry_Pi_2_3, J2 6P6C, J3 TC2030, SW1 SW_Push

Commit message: Getting ready for v0.3.0
Parts:
- removed TP1, TP2, TP3, TP4, TP5, TP6: TestPoint, TestPoint:TestPoint_THTPad_D1.0mm_Drill0.5mm, symbol cacophony-library:TestPoint
- added J5, J6: Conn_02x06_Odd_Even, Connector_PinHeader_2.54mm:PinHeader_2x06_P2.54mm_Vertical, symbol Connector_Generic:Conn_02x06_Odd_Even
- added R5, R6: 10k, Resistor_THT:R_Axial_DIN0207_L6.3mm_D2.5mm_P7.62mm_Horizontal, symbol Device:R
- added SW2, SW3, SW4: SW_Push, cacophony-library:SW_PUSH_6mm_11mmh, symbol cacophony-library:SW_Push
- added U1: HS96L03W2C03, cacophony-library:OLED-TH_L27.8-W27.2-P2.54_C9900033791, symbol cacophony-library:HS96L03W2C03
- J1: footprint cacophony-library:rpi-zero-throughhole-socket -> cacophony-library:rpi-3-hat
Connections:
- net GND: now also J5.3 (Pin_3), J5.9 (Pin_9), R5.2, R6.2, SW2.2, SW3.2, SW4.2, U1.1 (GND)
- net LED_B: now also J1.24 (~{CE0}/GPIO8); no longer J1.35 (GPIO19/MISO1)
- net LED_G: now also J1.26 (~{CE1}/GPIO7); no longer J1.37 (GPIO26)
- net LED_R: now also J1.23 (SCLK0/GPIO11); no longer J1.33 (PWM1/GPIO13)
- net EEPROM_~{WC}_TEST: now reaches J3.1
- net SDA_TEST: now reaches J3.2
- net SCL_TEST: now reaches J3.4
- net +3.3V: now reaches J1.1 (3V3), J1.17 (3V3)
- net +3.3V: now also J5.12 (Pin_12), J5.6 (Pin_6), U1.2 (VCC)
- net at J1.11 (GPIO17): now also JP1.2 (B)
- net GPIO18: now reaches J1.12 (GPIO18/PWM0)
- net GPIO18: now also J5.11 (Pin_11)
- net GPIO27: now reaches J1.13 (GPIO27)
- net GPIO27: now also J5.10 (Pin_10)
- net GPIO22: now reaches J1.15 (GPIO22)
- net GPIO22: now also J5.8 (Pin_8)
- net GPIO23: now reaches J1.16 (GPIO23)
- net GPIO23: now also J5.7 (Pin_7)
- net GPIO24: now reaches J1.18 (GPIO24)
- net GPIO24: now also J5.5 (Pin_5)
- net GPIO10: now reaches J1.19 (MOSI0/GPIO10)
- net GPIO10: now also J5.4 (Pin_4)
- net +5V: now reaches J1.2 (5V), J1.4 (5V)
- net GPIO9: now reaches J1.21 (MISO0/GPIO9)
- net GPIO9: now also J5.2 (Pin_2)
- net PROGRAM_CAMERA: now reaches J1.29 (GCLK1/GPIO5)
- net SDA: now reaches J1.3 (SDA/GPIO2)
- net SDA: now also J2.5, R5.1, U1.4 (SDA)
- net PROGRAM_TRAP: now reaches J1.32 (PWM0/GPIO12)
- net GPIO16: now reaches J1.36 (GPIO16)
- net GPIO16: now also J6.5 (Pin_5)
- net GPIO20: now reaches J1.38 (GPIO20/MOSI1)
- net GPIO20: now also J6.3 (Pin_3)
- net GPIO21: now reaches J1.40 (GPIO21/SCLK1)
- net GPIO21: now also J6.1 (Pin_1)
- net SCL: now reaches J1.5 (SCL/GPIO3)
- net SCL: now also J2.3, R6.1, U1.3 (SCL)
- net EEPROM_~{WC}: now reaches J1.7 (GCLK0/GPIO4)
- net EEPROM_~{WC}: now also J2.6
- net BUTTON renamed PROGRAM_BATTERY_BUTTON
- net PROGRAM_BATTERY_BUTTON: now also SW2.1; no longer SW1.1
- net RPI_RX renamed GPIO25
- net GPIO25: now also J5.1 (Pin_1); no longer JP1.2 (B)
- new net GPIO13: J1.33 (PWM1/GPIO13), J6.8 (Pin_8)
- new net GPIO19: J1.35 (GPIO19/MISO1), J6.6 (Pin_6)
- new net GPIO26: J1.37 (GPIO26), J6.4 (Pin_4)
- new net PROGRAM_BATTERY_FIRMWARE: SW4.1
- new net PROGRAM_CAMERA_EEPROM: SW1.1
- new net PROGRAM_TRAP_EEPROM: SW3.1
- no-connect marks 29 -> 2
Other:
- moved on the sheet: JP1, SW1
